File: postive12Vsupply.sch (KiCad schematic (older format))
At the start: 18 parts, among them U1 LT3959

Commit message: Named nets, made it use 2 inductors
Parts:
- removed L1: DRQ127-150, eaton:eaton_drq127, symbol coiltronics:DRQ127-150
- added L1, L4: SRP1265A-330M, bourns:bourns_srp1265a, symbol Device:L
Connections:
- net Earth: now also U1.1 (NC), U1.2 (NC), U1.3 (NC), U1.35 (NC), U1.36 (NC), U1.37 (NC), U1.38 (NC), L4.2
- net Vin2.5-24V: now also L1.1
- net SGND: now reaches C3.2, C4.2, C5.1, R3.2, R5.2, R7.2, U1.10 (SGND), U1.17 (GNDK), U1.29 (SGND), U1.8 (SYNC)
- net SGND: now also U1.11 (NC), U1.28 (NC)
- net SW: now reaches C6.1, U1.12 (SW), U1.15 (SW), U1.24 (SW), U1.27 (SW)
- net SW: now also U1.13 (NC), U1.14 (NC), U1.16 (NC), U1.23 (NC), U1.25 (NC), U1.26 (NC), L1.2
- net EN_UVLO: now reaches R4.2, R5.1, U1.34 (EN/UVLO)
- net FBX: now reaches R2.2, R3.1, U1.5 (FBX)
- net DIODE_IN: now reaches C6.2, D1.2 (A)
- net DIODE_IN: now also L4.1
Other:
- moved on the sheet: C6

Commit message: Layed out inductors,
Now just have to lay out resistors that configure the power supply
Parts:
- D1: footprint Package_TO_SOT_SMD:TO-252-2 -> (none)
Changed lines of the file:
@@
 	1    0    0    -1
-$EndComp
-$Comp
-L Device:D_Schottky D?
-U 1 1 5CB5D620
-P 6250 1350
-AR Path="/5CB5D620" Ref="D?"  Part="1"
-AR Path="/5CA65B33/5CB5D620" Ref="D1"  Part="1"
-F 0 "D1" H 6250 1566 50  0000 C CNN
-F 1 "VISHAY 6CWQ06FN" H 6250 1475 50  0000 C CNN
-F 2 "Package_TO_SOT_SMD:TO-252-2" H 6250 1350 50  0001 C CNN
-F 3 "~" H 6250 1350 50  0001 C CNN
-	1    6250 1350
-	-1   0    0    -1
 $EndComp
 Wire Wire Line
@@
 	6400 3000 6400 1350
 Connection ~ 4500 3000
-Connection ~ 6400 1350
 Text Notes 6700 1750 0    50   ~ 0
 high di/dt loop
@@
 Text Label 5500 1350 0    50   ~ 0
 DIODE_IN
+$Comp
+L Device:D_Schottky D1
+U 1 1 5CB26F32
+P 6250 1350
+F 0 "D1" H 6250 1134 50  0000 C CNN
+F 1 "VISHAY 6CWQ06FN" H 6250 1225 50  0000 C CNN
+F 2 "" H 6250 1350 50  0001 C CNN
+F 3 "~" H 6250 1350 50  0001 C CNN
+	1    6250 1350
+	-1   0    0    1
+$EndComp
+Connection ~ 6400 1350
 $EndSCHEMATC

Commit message: Use better footprint for TO-252 diode package
Parts:
- D1: footprint (none) -> generic:D_TO-252
Changed lines of the file:
@@
 F 0 "D1" H 6250 1134 50  0000 C CNN
 F 1 "VISHAY 6CWQ06FN" H 6250 1225 50  0000 C CNN
-F 2 "" H 6250 1350 50  0001 C CNN
+F 2 "generic:D_TO-252" H 6250 1350 50  0001 C CNN
 F 3 "~" H 6250 1350 50  0001 C CNN
 	1    6250 1350
